File: pcb/revC/karabas-nano-revC.kicad_pcb (KiCad board)
At the start: 2 copper layers, 101.6 x 99.7 mm, 148 parts, among them J1 DC 5V, J10 PWR, J2 TAPE IN/OUT, J3 A/V, J4 BUS, J5 KEYBOARD, J6 BUS, J7 JTAG, J8 KEYBOARD, J9 RGB, Q1 BC846B, SW1 RESET, SW10 8, SW11 9, SW12 0, SW13 Q, SW14 A, SW15 CS, SW16 W, SW17 S, SW18 Z, SW19 E, SW2 NMI, SW20 D, SW21 X, SW22 R, SW23 F, SW24 C, SW25 T, SW26 G, SW27 V, SW28 Y, SW29 H, SW3 1, SW30 B, SW31 U, SW32 J, SW33 N, SW34 I, SW35 K, SW36 M, SW37 O, SW38 L, SW39 SS, SW4 2, SW40 P, SW41 Enter, SW42 Space, SW5 3, SW6 4, SW7 5, SW8 6, SW9 7, U1 Z80, U13 LM1117-3.3, U2 27C512, U3 BS62LV1600, U4 ATmega8A-AU, U6 EPM3256ATC144, U7 MicroSD, U9 AD724, Y1 28MHz, Y2 XMHz, Y3 4.43MHz, Y4 20MHz

Commit message: final revision rev.C
Parts:
- added H5: MountingHole, MountingHole:MountingHole_2.5mm_Pad, F.Cu at (91.9, 126.5)
- added H6: MountingHole, MountingHole:MountingHole_2.5mm_Pad, F.Cu at (91.9, 147.3)
- added H7: MountingHole, MountingHole:MountingHole_2.5mm_Pad, F.Cu at (187.5, 126.5)
- added H8: MountingHole, MountingHole:MountingHole_2.5mm_Pad, F.Cu at (187.5, 147.3)
- added J11: AVR ISP, Connector_PinHeader_2.54mm:PinHeader_2x03_P2.54mm_Vertical, F.Cu at (137.7, 118.1)
- added R1: 10k, Resistor_SMD:R_0805_2012Metric, B.Cu at (179.8, 120.4)
- added R2: 10k, Resistor_SMD:R_0805_2012Metric, F.Cu at (179.8, 112.3)
- added R3: 10k, Resistor_SMD:R_0805_2012Metric, F.Cu at (175.8, 112.3)
- added REF**: KiCad-Logo2_12mm_SilkScreen, Symbol:KiCad-Logo2_12mm_SilkScreen, B.Cu at (110.2, 114.3)
- C14: footprint Capacitor_SMD:CP_Elec_5x4.4 -> Capacitor_Tantalum_SMD:CP_EIA-3528-21_Kemet-B_Pad1.50x2.35mm_HandSolder
- C9: footprint Capacitor_SMD:CP_Elec_8x6.5 -> Capacitor_Tantalum_SMD:CP_EIA-7343-31_Kemet-D_Pad2.25x2.55mm_HandSolder
- D10: value RED -> PWR
- D11: value GREEN -> SD
- D12: value GREEN -> MMC
- J10: footprint 1X02 -> Connector_PinHeader_2.54mm:PinHeader_1x02_P2.54mm_Vertical
- J4: footprint 1X16 -> Connector_PinHeader_2.54mm:PinHeader_1x16_P2.54mm_Vertical
- moved J8 4.96 mm to (97.0, 128.5)
- moved Y4 3.14 mm to (159.0, 98.6), turned to 0 degrees
- moved J10 2.54 mm to (180.3, 118.1), turned to 180 degrees
- moved J5 2.54 mm to (154.9, 118.1)
- turned J4 to 90 degrees
Connections:
- U4 pad 15: Net-(U4-Pad15) -> /AVR_MOSI
- U4 pad 16: Net-(U4-Pad16) -> /AVR_MISO
- U4 pad 17: Net-(U4-Pad17) -> /AVR_SCK
- U7 pad : (no net) -> GND
- U7 pad 10: (no net) -> GND
- U7 pad ~: (no net) -> GND
Routing:
- net /KA13: track 129.1 -> 182.0 mm, vias 12 -> 10
- net /AVR_MISO: track 0.00 -> 44.4 mm, vias 0 -> 1
- net /AVR_SCK: track 0.00 -> 42.6 mm, vias 0 -> 1
- net /AVR_MOSI: track 0.00 -> 41.4 mm, vias 0 -> 1
- net /VCCJP: track 23.4 -> 64.0 mm, vias 4 -> 5
- net /KB3: track 264.1 -> 241.7 mm, vias 5 -> 6
- net /KB4: track 244.5 -> 266.0 mm, vias 7 -> 8
- net ~RESET: track 187.4 -> 207.1 mm
- net GND: track 185.6 -> 192.9 mm, vias 163 -> 179
- net /KB2: track 252.0 -> 245.2 mm, vias 4 -> 5
- net /KB6: track 92.4 -> 86.3 mm
- net Net-(U4-Pad8): track 15.6 -> 21.7 mm
- net /AY_OUT_R: track 158.3 -> 152.3 mm
- net /KB7: track 95.3 -> 89.8 mm
- net /KB5: track 89.7 -> 84.3 mm
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Other:
- board text added: "A11 A10 A9 A12 A13 A8 A14 A15 RES TURBO"
- board text added: "BC1 SDC SDS CLK F28 A12 A8 A6 A4 A2 RFSH NMI BACK BREQ IOE RESET"
- board text added: "BDIR SDO SDI ROMCS CLKX A10 A13 A14 A5 A1 M1 WAIT INT MREQ IORQ D7 D4 D5 D2 VCC"
- board text added: "BEEP IO16 IO13 MAPC IORQ A11 A9 A15 A7 A0 A3 WR HALT NMI RD D0 D3 D6 D1 GND"
- board text added: "GND"
- board text added: "KB0 KB1 KB2 KB3 KB4 KB5"
- board text added: "MISO SCK RESET"
- board text added: "R G B S GND VCC"
- board text added: "VCC"
- board text added: "VCC MOSI GND"
