File: pcb/revC/karabas-nano-revC.sch (KiCad schematic (older format))
At the start: 148 parts, among them J1 DC 5V, J10 PWR, J2 TAPE IN/OUT, J3 A/V, J4 BUS, J5 KEYBOARD, J6 BUS, J7 JTAG, J8 KEYBOARD, J9 RGB, Q1 BC846B, SW1 RESET, SW10 8, SW11 9, SW12 0, SW13 Q, SW14 A, SW15 CS, SW16 W, SW17 S, SW18 Z, SW19 E, SW2 NMI, SW20 D, SW21 X, SW22 R, SW23 F, SW24 C, SW25 T, SW26 G, SW27 V, SW28 Y, SW29 H, SW3 1, SW30 B, SW31 U, SW32 J, SW33 N, SW34 I, SW35 K, SW36 M, SW37 O, SW38 L, SW39 SS, SW4 2, SW40 P, SW41 Enter, SW42 Space, SW5 3, SW6 4, SW7 5, SW8 6, SW9 7, U1 Z80, U13 LM1117-3.3, U2 27C512, U3 BS62LV1600, U4 ATmega8A-AU, U6 EPM3256ATC144, U7 MicroSD, U9 AD724, Y1 28MHz, Y2 XMHz, Y3 4.43MHz, Y4 20MHz

Commit message: final revision rev.C
Parts:
- added H? (x4): MountingHole, MountingHole:MountingHole_2.5mm_Pad, symbol Mechanical:MountingHole
- added J11: AVR ISP, Connector_PinHeader_2.54mm:PinHeader_2x03_P2.54mm_Vertical, symbol SparkFun-Connectors:AVR_SPI_PROG_3X22X3_LOCK
- added R1, R2, R3: 10k, Resistor_SMD:R_0805_2012Metric, symbol Device:R
- C14: footprint Capacitor_SMD:CP_Elec_5x4.4 -> Capacitor_Tantalum_SMD:CP_EIA-3528-21_Kemet-B_Pad1.50x2.35mm_HandSolder
- C9: footprint Capacitor_SMD:CP_Elec_8x6.5 -> Capacitor_Tantalum_SMD:CP_EIA-7343-31_Kemet-D_Pad2.25x2.55mm_HandSolder
- D10: value RED -> PWR
- D11: value GREEN -> SD
- D12: value GREEN -> MMC
- J10: footprint 1X02 -> Connector_PinHeader_2.54mm:PinHeader_1x02_P2.54mm_Vertical
- J4: footprint 1X16 -> Connector_PinHeader_2.54mm:PinHeader_1x16_P2.54mm_Vertical
Connections:
- net GND: now also J11.6 (GND), R1.2, R2.2, R3.2
- net MAGIC: now also R2.1
- net SPECIAL: now also R3.1
- net TURBO: now also R1.1
- net VCCJP: now also J11.2 (VCC)
- net ~RESET: now also J11.5 (RST)
- net AVR_MOSI: now reaches U4.15 (PB3)
- net AVR_MOSI: now also J11.4 (MOSI)
- net AVR_MISO: now reaches U4.16 (PB4)
- net AVR_MISO: now also J11.1 (MISO)
- net AVR_SCK: now reaches U4.17 (PB5)
- net AVR_SCK: now also J11.3 (SCK)
- no-connect marks 19 -> 16
Changed lines of the file:
@@
 EESchema Schematic File Version 4
-LIBS:karabas-nano-revB1-cache
 EELAYER 26 0
 EELAYER END
@@
 F 0 "C9" V 5205 8800 50  0000 C CNN
 F 1 "220uF" V 5114 8800 50  0000 C CNN
-F 2 "Capacitor_SMD:CP_Elec_8x6.5" H 4988 8650 50  0001 C CNN
+F 2 "Capacitor_Tantalum_SMD:CP_EIA-7343-31_Kemet-D_Pad2.25x2.55mm_HandSolder" H 4988 8650 50  0001 C CNN
 F 3 "~" H 4950 8800 50  0001 C CNN
 	1    4950 8800
@@
 F 0 "C14" H 3868 4046 50  0000 L CNN
 F 1 "10uF" H 3868 3955 50  0000 L CNN
-F 2 "Capacitor_SMD:CP_Elec_5x4.4" H 3788 3850 50  0001 C CNN
+F 2 "Capacitor_Tantalum_SMD:CP_EIA-3528-21_Kemet-B_Pad1.50x2.35mm_HandSolder" H 3788 3850 50  0001 C CNN
 F 3 "~" H 3750 4000 50  0001 C CNN
 	1    3750 4000
@@
 F 0 "J4" H 13422 7658 45  0000 R CNN
 F 1 "BUS" H 13422 7742 45  0000 R CNN
-F 2 "1X16" H 13700 8650 20  0001 C CNN
+F 2 "Connector_PinHeader_2.54mm:PinHeader_1x16_P2.54mm_Vertical" H 13700 8650 20  0001 C CNN
 F 3 "" H 13700 6950 50  0001 C CNN
 F 4 "XXX-00000" H 13633 8581 60  0001 C CNN "Field4"
@@
 NoConn ~ 7350 6300
 NoConn ~ 7350 6400
-NoConn ~ 7350 5000
-NoConn ~ 7350 4900
-NoConn ~ 7350 4800
 NoConn ~ 7350 4500
 NoConn ~ 6150 5300
@@
 P 15350 1800
 F 0 "D10" H 15300 2031 60  0000 C CNN
-F 1 "RED" H 15300 2031 60  0001 C CNN
+F 1 "PWR" H 15300 2031 60  0001 C CNN
 F 2 "digikey-footprints:0805" H 15550 2000 60  0001 L CNN
 F 3 "https://dammedia.osram.info/media/resource/hires/osram-dam-2493936/LG%20R971.pdf" H 15550 2100 60  0001 L CNN
@@
 P 15350 2200
 F 0 "D11" H 15300 2431 60  0000 C CNN
-F 1 "GREEN" H 15300 2431 60  0001 C CNN
+F 1 "SD" H 15300 2431 60  0001 C CNN
 F 2 "digikey-footprints:0805" H 15550 2400 60  0001 L CNN
 F 3 "https://dammedia.osram.info/media/resource/hires/osram-dam-2493888/LH%20R974.pdf" H 15550 2500 60  0001 L CNN
@@
 F 0 "J10" H 9022 8192 45  0000 R CNN
 F 1 "PWR" H 9022 8108 45  0000 R CNN
-F 2 "1X02" H 9250 8350 20  0001 C CNN
+F 2 "Connector_PinHeader_2.54mm:PinHeader_1x02_P2.54mm_Vertical" H 9250 8350 20  0001 C CNN
 F 3 "" H 9250 8100 50  0001 C CNN
 F 4 "XXX-00000" H 9022 8066 60  0001 R CNN "Field4"
@@
 P 15350 2550
 F 0 "D12" H 15300 2781 60  0000 C CNN
-F 1 "GREEN" H 15300 2781 60  0001 C CNN
+F 1 "MMC" H 15300 2781 60  0001 C CNN
 F 2 "digikey-footprints:0805" H 15550 2750 60  0001 L CNN
 F 3 "https://dammedia.osram.info/media/resource/hires/osram-dam-2493888/LH%20R974.pdf" H 15550 2850 60  0001 L CNN
@@
 	1    0    0    -1
 $EndComp
+Text Label 6950 4200 0    50   ~ 0
+VCCJP
+Text Label 9150 10150 0    50   ~ 0
+VCCJP
+$Comp
+L SparkFun-Connectors:AVR_SPI_PROG_3X22X3_LOCK J11
+U 1 1 5D678BEB
+P 13900 9050
+F 0 "J11" H 13900 9354 45  0000 C CNN
+F 1 "AVR ISP" H 13900 9270 45  0000 C CNN
+F 2 "Connector_PinHeader_2.54mm:PinHeader_2x03_P2.54mm_Vertical" H 13900 9350 20  0001 C CNN
+F 3 "" H 13900 9050 50  0001 C CNN
+F 4 "XXX-00000" H 13900 9281 60  0001 C CNN "Поле4"
+	1    13900 9050
+	1    0    0    -1
+$EndComp
+Entry Wire Line
+	14500 8950 14600 8850
+Entry Wire Line
+	14500 9050 14600 8950
+Entry Wire Line
+	14500 9150 14600 9050
+Entry Wire Line
+	12950 8850 13050 8950
+Entry Wire Line
+	12950 8950 13050 9050
+Entry Wire Line
+	12950 9050 13050 9150
 Wire Bus Line
-	14150 6500 14150 7650
+	12950 9250 14600 9250
+Wire Wire Line
+	13050 8950 13600 8950
+Wire Wire Line
+	13050 9050 13600 9050
+Wire Wire Line
+	13050 9150 13600 9150
+Wire Wire Line
+	14200 8950 14500 8950
+Wire Wire Line
+	14200 9050 14500 9050
+Wire Wire Line
+	14200 9150 14500 9150
+Text Label 13050 8950 0    50   ~ 0
+AVR_MISO
+Text Label 13050 9050 0    50   ~ 0
+AVR_SCK
+Text Label 13050 9150 0    50   ~ 0
+~RESET
+Text Label 14500 9150 2    50   ~ 0
+GND
+Text Label 14500 8950 2    50   ~ 0
+VCCJP
+Text Label 14500 9050 2    50   ~ 0
+AVR_MOSI
+Entry Wire Line
+	7900 4800 8000 4700
+Entry Wire Line
+	7900 4900 8000 4800
+Entry Wire Line
+	7900 5000 8000 4900
+Wire Wire Line
+	7350 4800 7900 4800
+Wire Wire Line
+	7350 4900 7900 4900
+Wire Wire Line
+	7350 5000 7900 5000
+Text Label 7900 5000 2    50   ~ 0
+AVR_SCK
+Text Label 7900 4900 2    50   ~ 0
+AVR_MISO
+Text Label 7900 4800 2    50   ~ 0
+AVR_MOSI
+$Comp
+L Device:R R1
+U 1 1 5E037A5E
+P 10700 8400
+F 0 "R1" V 10907 8400 50  0000 C CNN
+F 1 "10k" V 10816 8400 50  0000 C CNN
+F 2 "Resistor_SMD:R_0805_2012Metric" V 10630 8400 50  0001 C CNN
+F 3 "~" H 10700 8400 50  0001 C CNN
+	1    10700 8400
+	0    -1   -1   0
+$EndComp
+$Comp
+L Device:R R2
+U 1 1 5E1324F4
+P 10700 8700
+F 0 "R2" V 10907 8700 50  0000 C CNN
+F 1 "10k" V 10816 8700 50  0000 C CNN
+F 2 "Resistor_SMD:R_0805_2012Metric" V 10630 8700 50  0001 C CNN
+F 3 "~" H 10700 8700 50  0001 C CNN
+	1    10700 8700
+	0    -1   -1   0
+$EndComp
+$Comp
+L Device:R R3
+U 1 1 5E132679
+P 10700 9050
+F 0 "R3" V 10907 9050 50  0000 C CNN
+F 1 "10k" V 10816 9050 50  0000 C CNN
+F 2 "Resistor_SMD:R_0805_2012Metric" V 10630 9050 50  0001 C CNN
+F 3 "~" H 10700 9050 50  0001 C CNN
+	1    10700 9050
+	0    -1   -1   0
+$EndComp
+Entry Wire Line
+	10200 8950 10300 9050
+Entry Wire Line
+	10200 8600 10300 8700
+Entry Wire Line
+	10200 8300 10300 8400
+Wire Wire Line
+	10300 8400 10550 8400
+Wire Wire Line
+	10300 8700 10550 8700
+Wire Wire Line
+	10300 9050 10550 9050
+$Comp
+L power:GND #PWR0117
+U 1 1 5E520BEC
+P 10900 9100
+F 0 "#PWR0117" H 10900 8850 50  0001 C CNN
+F 1 "GND" H 10905 8927 50  0000 C CNN
+F 2 "" H 10900 9100 50  0001 C CNN
+F 3 "" H 10900 9100 50  0001 C CNN
+	1    10900 9100
+	1    0    0    -1
+$EndComp
+Wire Wire Line
+	10850 8400 10900 8400
+Wire Wire Line
+	10900 8400 10900 8700
+Wire Wire Line
+	10850 8700 10900 8700
+Connection ~ 10900 8700
+Wire Wire Line
+	10900 8700 10900 9050
+Wire Wire Line
+	10850 9050 10900 9050
 Wire Bus Line
-	10200 6500 10200 7750
+	14600 8850 14600 9250
+Wire Bus Line
+	14150 6500 14150 7650
 Wire Bus Line
 	750  3200 750  10850
@@
 	750  750  3450 750
 Wire Bus Line
+	10200 6500 10200 8950
+Wire Bus Line
 	10200 6500 11200 6500
 Wire Bus Line
@@
 	11200 6500 12950 6500
 Wire Bus Line
-	12950 6500 12950 8750
-Wire Bus Line
 	11200 6500 11200 8750
 Wire Bus Line
 	5500 750  5500 6050
 Wire Bus Line
+	12950 6500 12950 9250
+Wire Bus Line
 	8000 750  8000 6500
 Wire Bus Line
@@
 Wire Bus Line
 	8000 750  14100 750
-Text Label 6950 4200 0    50   ~ 0
-VCCJP
-Text Label 9150 10150 0    50   ~ 0
-VCCJP
+Connection ~ 10900 9050
+Wire Wire Line
+	10900 9050 10900 9100
+Text Label 10300 8400 0    50   ~ 0
+TURBO
+Text Label 10300 8700 0    50   ~ 0
+MAGIC
+Text Label 10300 9050 0    50   ~ 0
+SPECIAL
+$Comp
+L Mechanical:MountingHole H?
+U 1 1 5E81FCAC
+P 14850 9100
+F 0 "H?" H 14950 9146 50  0000 L CNN
+F 1 "MountingHole" H 14950 9055 50  0000 L CNN
+F 2 "MountingHole:MountingHole_2.5mm_Pad" H 14850 9100 50  0001 C CNN
+F 3 "~" H 14850 9100 50  0001 C CNN
+	1    14850 9100
+	1    0    0    -1
+$EndComp
+$Comp
+L Mechanical:MountingHole H?
+U 1 1 5E81FE7F
+P 14850 9300
+F 0 "H?" H 14950 9346 50  0000 L CNN
+F 1 "MountingHole" H 14950 9255 50  0000 L CNN
+F 2 "MountingHole:MountingHole_2.5mm_Pad" H 14850 9300 50  0001 C CNN
+F 3 "~" H 14850 9300 50  0001 C CNN
+	1    14850 9300
+	1    0    0    -1
+$EndComp
+$Comp
+L Mechanical:MountingHole H?
+U 1 1 5E81FF83
+P 14850 9500
+F 0 "H?" H 14950 9546 50  0000 L CNN
+F 1 "MountingHole" H 14950 9455 50  0000 L CNN
+F 2 "MountingHole:MountingHole_2.5mm_Pad" H 14850 9500 50  0001 C CNN
+F 3 "~" H 14850 9500 50  0001 C CNN
+	1    14850 9500
+	1    0    0    -1
+$EndComp
+$Comp
+L Mechanical:MountingHole H?
+U 1 1 5E82007D
+P 14850 9700
+F 0 "H?" H 14950 9746 50  0000 L CNN
+F 1 "MountingHole" H 14950 9655 50  0000 L CNN
+F 2 "MountingHole:MountingHole_2.5mm_Pad" H 14850 9700 50  0001 C CNN
+F 3 "~" H 14850 9700 50  0001 C CNN
+	1    14850 9700
+	1    0    0    -1
+$EndComp
 $EndSCHEMATC

Commit message: latest schematics
Parts:
- gave numbers to parts that had none: 4
Changed lines of the file:
@@
 SPECIAL
 $Comp
-L Mechanical:MountingHole H?
+L Mechanical:MountingHole H5
 U 1 1 5E81FCAC
 P 14850 9100
-F 0 "H?" H 14950 9146 50  0000 L CNN
+F 0 "H5" H 14950 9146 50  0000 L CNN
 F 1 "MountingHole" H 14950 9055 50  0000 L CNN
 F 2 "MountingHole:MountingHole_2.5mm_Pad" H 14850 9100 50  0001 C CNN
@@
 $EndComp
 $Comp
-L Mechanical:MountingHole H?
+L Mechanical:MountingHole H6
 U 1 1 5E81FE7F
 P 14850 9300
-F 0 "H?" H 14950 9346 50  0000 L CNN
+F 0 "H6" H 14950 9346 50  0000 L CNN
 F 1 "MountingHole" H 14950 9255 50  0000 L CNN
 F 2 "MountingHole:MountingHole_2.5mm_Pad" H 14850 9300 50  0001 C CNN
@@
 $EndComp
 $Comp
-L Mechanical:MountingHole H?
+L Mechanical:MountingHole H7
 U 1 1 5E81FF83
 P 14850 9500
-F 0 "H?" H 14950 9546 50  0000 L CNN
+F 0 "H7" H 14950 9546 50  0000 L CNN
 F 1 "MountingHole" H 14950 9455 50  0000 L CNN
 F 2 "MountingHole:MountingHole_2.5mm_Pad" H 14850 9500 50  0001 C CNN
@@
 $EndComp
 $Comp
-L Mechanical:MountingHole H?
+L Mechanical:MountingHole H8
 U 1 1 5E82007D
 P 14850 9700
-F 0 "H?" H 14950 9746 50  0000 L CNN
+F 0 "H8" H 14950 9746 50  0000 L CNN
 F 1 "MountingHole" H 14950 9655 50  0000 L CNN
 F 2 "MountingHole:MountingHole_2.5mm_Pad" H 14850 9700 50  0001 C CNN
