File: pcb/revD/karabas-nano-revD.kicad_pcb (KiCad board)
At the start: 2 copper layers, 101.6 x 99.7 mm, 153 parts, among them J1 DC 5V, J10 PWR, J11 AVR ISP, J2 TAPE IN/OUT, J3 A/V, J4 BUS, J5 KEYBOARD, J6 BUS, J7 JTAG, J9 RGB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

Commit message: latest fixes
Other:
- board text added: "J2 TAPE"
- board text added: "J3 A/V"
- board text added: "Y1 28MHz"
- board text added: "Y2 XMHz"
- board text added: "Y3"
- board text added: "Y4 20MHz"
