File: pcb/revH/karabas-nano-revH.sch (KiCad schematic (older format))
At the start: 158 parts, among them J1 USB_B_Micro, J10 PWR, J11 AVR ISP, J2 TAPE IN/OUT, J3 A/V, J4 BUS, J5 KEYBOARD, J6 BUS, J7 JTAG, J9 RGB, Q2 BC856, SW1 RESET, SW10 8, SW11 9, SW12 0, SW13 Q, SW14 A, SW15 CS, SW16 W, SW17 S, SW18 Z, SW19 E, SW2 NMI, SW20 D, SW21 X, SW22 R, SW23 F, SW24 C, SW25 T, SW26 G, SW27 V, SW28 Y, SW29 H, SW3 1, SW30 B, SW31 U, SW32 J, SW33 N, SW34 I, SW35 K, SW36 M, SW37 O, SW38 L, SW39 SS, SW4 2, SW40 P, SW41 Enter, SW42 Space, SW5 3, SW6 4, SW7 5, SW8 6, SW9 7, U1 Z80, U13 LM1117-3.3, U2 39F040, U3 CY62167ELL, U4 ATmega8A-AU, U5 ESP-12E, U6 EPM3256ATC144, U7 MicroSD, U8 LM311, U9 AD724, Y1 28MHz, Y3 4.43MHz, Y4 20MHz

Commit message: Added 3.3/5v selectors for memory and generator
Parts:
- added C1: 100nF, Capacitor_SMD:C_0805_2012Metric, symbol Device:C
- added JP5, JP6: 3/5V, Jumper:SolderJumper-3_P1.3mm_Open_RoundedPad1.0x1.5mm, symbol Jumper:SolderJumper_3_Open
Connections:
- net +3V3: now also C1.2, JP5.1 (A), JP6.1 (A); no longer Y1.1 (EN), Y1.4 (VCC)
- net GND: now also C1.1
- net VCC: now also JP5.3 (B), JP6.3 (B); no longer U3.12 (CE2), U3.37 (VCC)
- new net: JP5.2 (C), Y1.1 (EN), Y1.4 (VCC)
- new net: JP6.2 (C), U3.12 (CE2), U3.37 (VCC)
Other:
- moved on the sheet: Y1
Changed lines of the file:
@@
 $EndComp
 Entry Wire Line
-	3350 3550 3450 3450
-Text Label 3150 3550 0    50   ~ 0
+	3350 3850 3450 3750
+Text Label 3150 3850 0    50   ~ 0
 CLK28
 Entry Wire Line
@@
 L SparkFun-Clocks:OSCILLATORSMD-7X5-4PAD Y1
 U 1 1 5D58AEC5
-P 1950 3650
-F 0 "Y1" H 1950 4004 45  0000 C CNN
-F 1 "28MHz" H 1950 3920 45  0000 C CNN
-F 2 "Oscillator:Oscillator_SMD_EuroQuartz_XO91-4Pin_7.0x5.0mm" H 1950 4000 20  0001 C CNN
-F 3 "" H 1950 3650 50  0001 C CNN
-F 4 "XXX-00000" H 1950 3931 60  0001 C CNN "Field4"
-	1    1950 3650
+P 2550 3950
+F 0 "Y1" H 2550 4304 45  0000 C CNN
+F 1 "28MHz" H 2550 4220 45  0000 C CNN
+F 2 "Oscillator:Oscillator_SMD_EuroQuartz_XO91-4Pin_7.0x5.0mm" H 2550 4300 20  0001 C CNN
+F 3 "" H 2550 3950 50  0001 C CNN
+F 4 "XXX-00000" H 2550 4231 60  0001 C CNN "Field4"
+	1    2550 3950
 	1    0    0    -1
 $EndComp
 Wire Wire Line
-	2350 3550 3350 3550
+	2950 3850 3350 3850
 $Comp
 L power:GND #PWR0108
 U 1 1 5F1790C3
-P 2450 3750
-F 0 "#PWR0108" H 2450 3500 50  0001 C CNN
-F 1 "GND" H 2455 3577 50  0000 C CNN
-F 2 "" H 2450 3750 50  0001 C CNN
-F 3 "" H 2450 3750 50  0001 C CNN
-	1    2450 3750
+P 3050 4050
+F 0 "#PWR0108" H 3050 3800 50  0001 C CNN
+F 1 "GND" H 3055 3877 50  0000 C CNN
+F 2 "" H 3050 4050 50  0001 C CNN
+F 3 "" H 3050 4050 50  0001 C CNN
+	1    3050 4050
 	1    0    0    -1
 $EndComp
 Wire Wire Line
-	2350 3750 2450 3750
+	2950 4050 3050 4050
 $Comp
 L power:+3V3 #PWR0115
 U 1 1 5F35EEC4
-P 1450 3550
-F 0 "#PWR0115" H 1450 3400 50  0001 C CNN
-F 1 "+3V3" H 1465 3723 50  0000 C CNN
-F 2 "" H 1450 3550 50  0001 C CNN
-F 3 "" H 1450 3550 50  0001 C CNN
-	1    1450 3550
+P 1400 3600
+F 0 "#PWR0115" H 1400 3450 50  0001 C CNN
+F 1 "+3V3" H 1415 3773 50  0000 C CNN
+F 2 "" H 1400 3600 50  0001 C CNN
+F 3 "" H 1400 3600 50  0001 C CNN
+	1    1400 3600
 	1    0    0    -1
 $EndComp
 Wire Wire Line
-	1450 3550 1550 3550
+	2050 3850 2150 3850
 Wire Wire Line
-	1550 3750 1450 3750
+	2150 4050 2050 4050
 Wire Wire Line
-	1450 3750 1450 3550
-Connection ~ 1450 3550
+	2050 4050 2050 3850
 Entry Wire Line
 	12950 7950 13050 8050
@@
 Wire Wire Line
 	6100 3750 6200 3750
-Entry Wire Line
-	5500 3750 5600 3850
-Wire Wire Line
-	6200 3850 5600 3850
-Text Label 5600 3850 0    50   ~ 0
-VCC
-Entry Wire Line
-	7900 3650 8000 3550
-Wire Wire Line
-	7300 3650 7900 3650
-Text Label 7900 3650 2    50   ~ 0
-VCC
 $Comp
 L Transistor_BJT:BC856 Q2
@@
 Wire Wire Line
 	3050 7650 2800 7650
+Connection ~ 2800 7650
+$Comp
+L Jumper:SolderJumper_3_Open JP5
+U 1 1 658800E6
+P 1700 3650
+F 0 "JP5" H 1700 3855 50  0000 C CNN
+F 1 "3/5V" H 1700 3764 50  0000 C CNN
+F 2 "Jumper:SolderJumper-3_P1.3mm_Open_RoundedPad1.0x1.5mm" H 1700 3650 50  0001 C CNN
+F 3 "~" H 1700 3650 50  0001 C CNN
+	1    1700 3650
+	1    0    0    -1
+$EndComp
+$Comp
+L power:VCC #PWR0154
+U 1 1 65A76817
+P 2000 3600
+F 0 "#PWR0154" H 2000 3450 50  0001 C CNN
+F 1 "VCC" H 2017 3773 50  0000 C CNN
+F 2 "" H 2000 3600 50  0001 C CNN
+F 3 "" H 2000 3600 50  0001 C CNN
+	1    2000 3600
+	1    0    0    -1
+$EndComp
+Wire Wire Line
+	1400 3600 1400 3650
+Wire Wire Line
+	1400 3650 1500 3650
+Wire Wire Line
+	1900 3650 2000 3650
+Wire Wire Line
+	2000 3650 2000 3600
+Wire Wire Line
+	1700 3800 1700 3850
+Wire Wire Line
+	1700 3850 2050 3850
+Connection ~ 2050 3850
+$Comp
+L Jumper:SolderJumper_3_Open JP6
+U 1 1 65D6172D
+P 7650 3350
+F 0 "JP6" H 7650 3555 50  0000 C CNN
+F 1 "3/5V" H 7650 3464 50  0000 C CNN
+F 2 "Jumper:SolderJumper-3_P1.3mm_Open_RoundedPad1.0x1.5mm" H 7650 3350 50  0001 C CNN
+F 3 "~" H 7650 3350 50  0001 C CNN
+	1    7650 3350
+	1    0    0    -1
+$EndComp
+$Comp
+L power:+3V3 #PWR0155
+U 1 1 65D65016
+P 7450 3200
+F 0 "#PWR0155" H 7450 3050 50  0001 C CNN
+F 1 "+3V3" H 7465 3373 50  0000 C CNN
+F 2 "" H 7450 3200 50  0001 C CNN
+F 3 "" H 7450 3200 50  0001 C CNN
+	1    7450 3200
+	1    0    0    -1
+$EndComp
+$Comp
+L power:VCC #PWR0156
+U 1 1 65D69206
+P 7850 3200
+F 0 "#PWR0156" H 7850 3050 50  0001 C CNN
+F 1 "VCC" H 7867 3373 50  0000 C CNN
+F 2 "" H 7850 3200 50  0001 C CNN
+F 3 "" H 7850 3200 50  0001 C CNN
+	1    7850 3200
+	1    0    0    -1
+$EndComp
+Wire Wire Line
+	7300 3650 7650 3650
+Wire Wire Line
+	7650 3650 7650 3500
+Wire Wire Line
+	7450 3350 7450 3200
+Wire Wire Line
+	7850 3350 7850 3200
+Wire Wire Line
+	6200 3850 6200 4000
+Wire Wire Line
+	6200 4000 7650 4000
+Wire Wire Line
+	7650 4000 7650 3650
 Wire Bus Line
 	14600 8850 14600 9250
@@
 	11200 6500 11200 8750
 Wire Bus Line
-	12950 6500 12950 9250
-Wire Bus Line
 	5500 750  5500 4400
 Wire Bus Line
+	12950 6500 12950 9250
+Wire Bus Line
 	8000 750  8000 6500
 Wire Bus Line
@@
 Wire Bus Line
 	8000 750  13850 750
-Connection ~ 2800 7650
+Connection ~ 7650 3650
+$Comp
+L Device:C C1
+U 1 1 6615D0B7
+P 7350 9450
+F 0 "C1" H 7235 9404 50  0000 R CNN
+F 1 "100nF" H 7235 9495 50  0000 R CNN
+F 2 "Capacitor_SMD:C_0805_2012Metric" H 7388 9300 50  0001 C CNN
+F 3 "~" H 7350 9450 50  0001 C CNN
+	1    7350 9450
+	-1   0    0    1
+$EndComp
+$Comp
+L power:+3V3 #PWR0157
+U 1 1 661725BB
+P 7350 9300
+F 0 "#PWR0157" H 7350 9150 50  0001 C CNN
+F 1 "+3V3" H 7365 9473 50  0000 C CNN
+F 2 "" H 7350 9300 50  0001 C CNN
+F 3 "" H 7350 9300 50  0001 C CNN
+	1    7350 9300
+	1    0    0    -1
+$EndComp
+$Comp
+L power:GND #PWR0158
+U 1 1 66173AFC
+P 7350 9600
+F 0 "#PWR0158" H 7350 9350 50  0001 C CNN
+F 1 "GND" H 7355 9427 50  0000 C CNN
+F 2 "" H 7350 9600 50  0001 C CNN
+F 3 "" H 7350 9600 50  0001 C CNN
+	1    7350 9600
+	1    0    0    -1
+$EndComp
 $EndSCHEMATC
