File: pcb/revI/karabas-nano-revI.kicad_pcb (KiCad board)
At the start: 2 copper layers, 99.6 x 99.6 mm, 159 parts, among them J1 USB_B_Micro, J10 PWR, J11 AVR ISP, J2 TAPE IN/OUT, J3 A/V, J4 BUS, J5 KEYBOARD, J6 BUS, J7 JTAG, J8 AVR ISP, J9 RGB, Q2 BC856, SW1 RESET, SW10 8, SW11 9, SW12 0, SW13 Q, SW14 A, SW15 CS, SW16 W, SW17 S, SW18 Z, SW19 E, SW2 NMI, SW20 D, SW21 X, SW22 R, SW23 F, SW24 C, SW25 T, SW26 G, SW27 V, SW28 Y, SW29 H, SW3 1, SW30 B, SW31 U, SW32 J, SW33 N, SW34 I, SW35 K, SW36 M, SW37 O, SW38 L, SW39 SS, SW4 2, SW40 P, SW41 Enter, SW42 Space, SW5 3, SW6 4, SW7 5, SW8 6, SW9 7, U1 Z80, U10 ATmega8A-AU, U13 1117-3.3, U2 39F040, U3 CY62167ELL, U4 ATmega8A-AU, U5 ESP-12E, U6 EPM3256ATC144, U7 MicroSD, U8 LM311, U9 AD724, Y1 28MHz, Y3 4.43MHz

Commit message: upload final pcb rev.I files
Parts:
- U10, U4: value ATmega8A-AU -> ATmega88
Routing:
- net GND: track 275.3 -> 276.7 mm, vias 374 -> 376
- net /AY_OUT_R: track 124.8 -> 125.7 mm
- net KB2: track 209.8 -> 210.4 mm
- net /IO16: track 75.9 -> 75.3 mm
- net /~SD_CS: track 118.2 -> 117.6 mm
- net /SD_DI: track 108.0 -> 107.4 mm
- net /SD_CLK: track 104.5 -> 103.9 mm
- net /SD_DO: track 108.6 -> 108.0 mm
Other:
- board text added: "Rev.I"
- board text removed: "Rev.I-WIP"
