File: pcb/revI/karabas-nano-revI.kicad_sch (KiCad schematic)
At the start: 158 parts, among them J1 USB_B_Micro, J10 PWR, J11 AVR ISP, J2 TAPE IN/OUT, J3 A/V, J4 BUS, J5 KEYBOARD, J6 BUS, J7 JTAG, J8 AVR ISP, J9 RGB, Q2 BC856, SW1 RESET, SW10 8, SW11 9, SW12 0, SW13 Q, SW14 A, SW15 CS, SW16 W, SW17 S, SW18 Z, SW19 E, SW2 NMI, SW20 D, SW21 X, SW22 R, SW23 F, SW24 C, SW25 T, SW26 G, SW27 V, SW28 Y, SW29 H, SW3 1, SW30 B, SW31 U, SW32 J, SW33 N, SW34 I, SW35 K, SW36 M, SW37 O, SW38 L, SW39 SS, SW4 2, SW40 P, SW41 Enter, SW42 Space, SW5 3, SW6 4, SW7 5, SW8 6, SW9 7, U1 Z80, U10 ATmega8A-AU, U13 1117-3.3, U2 39F040, U3 CY62167ELL, U4 ATmega8A-AU, U5 ESP-12E, U6 EPM3256ATC144, U7 MicroSD, U8 LM311, U9 AD724, Y1 28MHz, Y3 4.43MHz

Commit message: upload final pcb rev.I files
Parts:
- U10, U4: value ATmega8A-AU -> ATmega88
Changed lines of the file:
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@@
     (in_bom yes) (on_board yes)
     (property "Reference" "U4" (id 0) (at 445.77 23.9776 0))
-    (property "Value" "ATmega8A-AU" (id 1) (at 445.77 26.289 0))
+    (property "Value" "ATmega88" (id 1) (at 445.77 26.289 0))
     (property "Footprint" "Package_QFP:TQFP-32_7x7mm_P0.8mm" (id 2) (at 445.77 64.135 0)
       (effects (font (size 1.27 1.27) italic) hide)
@@
     (in_bom yes) (on_board yes)
     (property "Reference" "U10" (id 0) (at 445.77 110.3376 0))
-    (property "Value" "ATmega8A-AU" (id 1) (at 445.77 112.649 0))
+    (property "Value" "ATmega88" (id 1) (at 445.77 112.649 0))
     (property "Footprint" "Package_QFP:TQFP-32_7x7mm_P0.8mm" (id 2) (at 445.77 150.495 0)
       (effects (font (size 1.27 1.27) italic) hide)
@@
     )
     (path "/00000000-0000-0000-0000-00006dd369c8"
-      (reference "U4") (unit 1) (value "ATmega8A-AU") (footprint "Package_QFP:TQFP-32_7x7mm_P0.8mm")
+      (reference "U4") (unit 1) (value "ATmega88") (footprint "Package_QFP:TQFP-32_7x7mm_P0.8mm")
     )
     (path "/00000000-0000-0000-0000-00005edb9366"
@@
     )
     (path "/5a8a6b05-a06a-4ba5-bc41-917030dafdc3"
-      (reference "U10") (unit 1) (value "ATmega8A-AU") (footprint "Package_QFP:TQFP-32_7x7mm_P0.8mm")
+      (reference "U10") (unit 1) (value "ATmega88") (footprint "Package_QFP:TQFP-32_7x7mm_P0.8mm")
     )
     (path "/00000000-0000-0000-0000-00005f242673"

Commit message: Updated 3d models on revI board
Connections:
- net ~BTN_NMI renamed ~{BTN_NMI}
- net ~BUSACK renamed ~{BUSACK}
- net ~BUSREQ renamed ~{BUSREQ}
- net ~BUS_IORQGE renamed ~{BUS_IORQGE}
- net ~BUS_ROMCS renamed ~{BUS_ROMCS}
- net ~HALT renamed ~{HALT}
- net ~INT renamed ~{INT}
- net ~IORQ renamed ~{IORQ}
- net ~M1 renamed ~{M1}
- net ~MRD renamed ~{MRD}
- net ~MREQ renamed ~{MREQ}
- net ~MWR renamed ~{MWR}
- net ~NMI renamed ~{NMI}
- net ~RD renamed ~{RD}
- net ~RESET renamed ~{RESET}
- net ~RFSH renamed ~{RFSH}
- net ~ROMCS renamed ~{ROMCS}
- net ~ROM_WE renamed ~{ROM_WE}
- net ~SD_CS renamed ~{SD_CS}
- net ~WAIT renamed ~{WAIT}
- net ~WR renamed ~{WR}
Other:
- title: (none) -> Karabas Nano
